File: esp01-1/esp-01.kicad_pcb (KiCad board)
At the start: 2 copper layers, 99.5 x 46.7 mm, 21 parts, among them P1 USB_B, SW1 Reset, SW2 Bootloader, U1 ESP-01V090, U2 LT1761-3.3, U3 MCP2200, Y1 CRYSTAL_SMD

Commit message: Reworked the esp-01 board routing
Parts:
- removed the Y1 at (77.5, 137.2)
- added C3: 4.7nF, Capacitors_ThroughHole:C_Disc_D6_P5, F.Cu at (79.6, 223.7)
- added R10: 1M, Resistors_ThroughHole:Resistor_Horizontal_RM10mm, F.Cu at (84.4, 223.7)
- added Y1: CRYSTAL_SMD, Resistors_SMD:Resonator_3.2x1.3mm, F.Cu at (0.00, 0.00)
- added Y1: CRYSTAL_SMD, cdtx:Resonator_3.2x1.3mm, F.Cu at (95.5, 213.4)
- C1: moved to B.Cu
- R1, R2, R3, R4, R7, R8: footprint Resistors_SMD:R_0805 -> Resistors_ThroughHole:Resistor_Horizontal_RM10mm
- R5, R9: footprint Resistors_SMD:R_0805 -> Resistors_SMD:R_0603
- R6: footprint Resistors_SMD:R_0805 -> Resistors_SMD:R_0603; moved to B.Cu
- SW1, SW2: footprint Buttons_Switches_SMD:SW_SPST_B3S-1000 -> Buttons_Switches_ThroughHole:SW_PUSH_SMALL
- moved P1 85.7 mm to (87.3, 214.6), turned to 180 degrees
- moved R7 84.6 mm to (129.3, 220.9)
- moved D3 82.1 mm to (78.7, 230.3)
- moved C1 81.4 mm to (126.1, 202.2), turned to 180 degrees
- moved D2 80.9 mm to (85.0, 230.3)
- moved R5 80.8 mm to (126.4, 227.7), turned to 180 degrees
- moved U2 80.1 mm to (76.0, 202.6)
- moved D1 80.1 mm to (90.8, 230.3)
- moved R8 79.9 mm to (125.6, 220.9), turned to 90 degrees
- moved SW1 78.6 mm to (119.1, 230.2)
- moved R9 78.2 mm to (111.3, 232.5)
- moved SW2 77.8 mm to (103.6, 230.2)
- moved R1 76.7 mm to (111.5, 222.4), turned to 90 degrees
- moved R3 72.6 mm to (101.1, 212.4)
- moved R4 70.6 mm to (92.7, 208.9)
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Routing:
- net GND: track 227.6 -> 29.8 mm, vias 4 -> 0
- net /usb_cfg: track 105.2 -> 19.2 mm
- net Net-(R5-Pad2): track 31.2 -> 112.3 mm
- net /USBD+: track 86.9 -> 23.5 mm, vias 2 -> 0
- net /USBD-: track 63.1 -> 22.8 mm, vias 2 -> 0
- net /usb_tx: track 35.3 -> 6.74 mm
- net Net-(U1-Pad8): track 49.8 -> 26.4 mm, vias 2 -> 1
- net +3V3: track 166.4 -> 183.3 mm, vias 0 -> 2
- net /usb_rx: track 23.4 -> 6.49 mm
- net Net-(D3-Pad2): track 6.06 -> 20.9 mm
- net Net-(D2-Pad2): track 7.33 -> 20.4 mm
- net Net-(D1-Pad2): track 6.43 -> 19.0 mm
- net Net-(C3-Pad1): track 0.00 -> 12.2 mm
- net Net-(R7-Pad2): track 3.38 -> 12.0 mm
- net Net-(U1-Pad1): track 21.9 -> 14.0 mm
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Other:
- board size 99.5 x 46.7 mm -> 64.1 x 46.7 mm
- net class Default: trace_width 0.4 -> 0.5; via_drill 1 -> 0.8
- rule via_min_drill: 0.508 -> 0.8
- rule via_min_size: 0.889 -> 2
- board text added: "PROG"
- board text added: "RESET"

Commit message: Removed unwanted footprint
Parts:
- removed the Y1 at (0.00, 0.00)
Changed lines of the file:
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@@
     (tracks 168)
     (zones 0)
-    (modules 24)
+    (modules 23)
     (nets 31)
   )
@@
       (net 7 "Net-(U1-Pad8)"))
   )
-  (module Resistors_SMD:Resonator_3.2x1.3mm (layer F.Cu)
-    (at 0 0)
-    (descr "Murata CSTCC8M00G53-R0; 8MHz resonator, SMD, 0.5+0.3%; Farnell (Element 14) #1170435")
-    (tags resonator)
-    (attr smd)
-    (fp_text reference Y1 (at 1.82 -1.91) (layer F.SilkS)
-      (effects (font (size 1 1) (thickness 0.15)))
-    )
-    (fp_text value CRYSTAL_SMD (at 1.93 2.9) (layer F.Fab)
-      (effects (font (size 1 1) (thickness 0.15)))
-    )
-    (fp_line (start 3.2 1.3) (end 3.2 0) (layer F.SilkS) (width 0.15))
-    (fp_line (start 0 0) (end 0 1.3) (layer F.SilkS) (width 0.15))
-    (fp_line (start 0 0) (end 3.2 0) (layer F.SilkS) (width 0.15))
-    (fp_line (start 3.2 1.3) (end 0 1.3) (layer F.SilkS) (width 0.15))
-    (pad 1 smd rect (at 2.66 0.64) (size 0.5 1.3) (layers F.Cu F.Paste F.Mask))
-    (pad 1 smd rect (at 1.6 0.64) (size 0.5 1.3) (layers F.Cu F.Paste F.Mask))
-    (pad 1 smd rect (at 0.51 0.63) (size 0.5 1.3) (layers F.Cu F.Paste F.Mask))
-  )
   (module cdtx:Resonator_3.2x1.3mm (layer F.Cu)
