File: esp01-1/esp-01.sch (KiCad schematic (older format))
At the start: 21 parts, among them P1 USB_B, SW1 Reset, SW2 Bootloader, U1 ESP-01V090, U2 LT1761-3.3, U3 MCP2200, Y1 CRYSTAL_SMD

Commit message: Reworked the esp-01 board routing
Parts:
- added C3: 4.7nF, Capacitors_ThroughHole:C_Disc_D6_P5, symbol C
- added R10: 1M, Resistors_ThroughHole:Resistor_Horizontal_RM10mm, symbol R
- R1, R2, R3, R4, R7, R8: footprint Resistors_SMD:R_0805 -> Resistors_ThroughHole:Resistor_Horizontal_RM10mm
- R5, R6, R9: footprint Resistors_SMD:R_0805 -> Resistors_SMD:R_0603
- SW1, SW2: footprint Buttons_Switches_SMD:SW_SPST_B3S-1000 -> Buttons_Switches_ThroughHole:SW_PUSH_SMALL
- Y1: footprint Crystals:Resonator_7.2x3mm -> cdtx:Resonator_3.2x1.3mm
Connections:
- wire segments 77 -> 85
Changed lines of the file:
@@
 F 0 "Y1" H 3300 2750 50  0000 C CNN
 F 1 "CRYSTAL_SMD" H 3400 2550 50  0000 L CNN
-F 2 "Crystals:Resonator_7.2x3mm" H 3300 2650 50  0001 C CNN
+F 2 "cdtx:Resonator_3.2x1.3mm" H 3300 2650 50  0001 C CNN
 F 3 "" H 3300 2650 50  0000 C CNN
 	1    3300 2650
@@
 F 0 "R1" H 2630 2870 50  0000 L CNN
 F 1 "10K" H 2630 2810 50  0000 L CNN
-F 2 "Resistors_SMD:R_0805" H 2600 2850 50  0001 C CNN
+F 2 "Resistors_ThroughHole:Resistor_Horizontal_RM10mm" H 2600 2850 50  0001 C CNN
 F 3 "" H 2600 2850 50  0000 C CNN
 	1    2600 2850
@@
 F 0 "R2" H 1330 3920 50  0000 L CNN
 F 1 "220R" H 1330 3860 50  0000 L CNN
-F 2 "Resistors_SMD:R_0805" H 1300 3900 50  0001 C CNN
+F 2 "Resistors_ThroughHole:Resistor_Horizontal_RM10mm" H 1300 3900 50  0001 C CNN
 F 3 "" H 1300 3900 50  0000 C CNN
 	1    1300 3900
@@
 F 0 "R3" H 1680 3920 50  0000 L CNN
 F 1 "220R" H 1680 3860 50  0000 L CNN
-F 2 "Resistors_SMD:R_0805" H 1650 3900 50  0001 C CNN
+F 2 "Resistors_ThroughHole:Resistor_Horizontal_RM10mm" H 1650 3900 50  0001 C CNN
 F 3 "" H 1650 3900 50  0000 C CNN
 	1    1650 3900
@@
 F 0 "R8" H 8330 4670 50  0000 L CNN
 F 1 "10K" H 8330 4610 50  0000 L CNN
-F 2 "Resistors_SMD:R_0805" H 8300 4650 50  0001 C CNN
+F 2 "Resistors_ThroughHole:Resistor_Horizontal_RM10mm" H 8300 4650 50  0001 C CNN
 F 3 "" H 8300 4650 50  0000 C CNN
 	1    8300 4650
@@
 F 0 "SW2" H 8450 5400 50  0000 C CNN
 F 1 "Bootloader" H 8350 5200 50  0000 L CNN
-F 2 "Buttons_Switches_SMD:SW_SPST_B3S-1000" H 8300 5500 50  0001 C CNN
+F 2 "Buttons_Switches_ThroughHole:SW_PUSH_SMALL" H 8300 5500 50  0001 C CNN
 F 3 "" H 8300 5500 50  0000 C CNN
 	1    8300 5300
@@
 F 0 "R7" H 7830 4670 50  0000 L CNN
 F 1 "10K" H 7830 4610 50  0000 L CNN
-F 2 "Resistors_SMD:R_0805" H 7800 4650 50  0001 C CNN
+F 2 "Resistors_ThroughHole:Resistor_Horizontal_RM10mm" H 7800 4650 50  0001 C CNN
 F 3 "" H 7800 4650 50  0000 C CNN
 	1    7800 4650
@@
 F 0 "R6" H 4980 4920 50  0000 L CNN
 F 1 "0" H 4980 4860 50  0000 L CNN
-F 2 "Resistors_SMD:R_0805" H 4950 4900 50  0001 C CNN
+F 2 "Resistors_SMD:R_0603" H 4950 4900 50  0001 C CNN
 F 3 "" H 4950 4900 50  0000 C CNN
 	1    4950 4900
@@
 F 0 "R9" H 8330 5620 50  0000 L CNN
 F 1 "100R" H 8330 5560 50  0000 L CNN
-F 2 "Resistors_SMD:R_0805" H 8300 5600 50  0001 C CNN
+F 2 "Resistors_SMD:R_0603" H 8300 5600 50  0001 C CNN
 F 3 "" H 8300 5600 50  0000 C CNN
 	1    8300 5600
@@
 F 0 "R5" H 4580 6220 50  0000 L CNN
 F 1 "10K" H 4580 6160 50  0000 L CNN
-F 2 "Resistors_SMD:R_0805" H 4550 6200 50  0001 C CNN
+F 2 "Resistors_SMD:R_0603" H 4550 6200 50  0001 C CNN
 F 3 "" H 4550 6200 50  0000 C CNN
 	1    4550 6200
@@
 F 0 "SW1" H 4700 6850 50  0000 C CNN
 F 1 "Reset" H 4450 6650 50  0000 L CNN
-F 2 "Buttons_Switches_SMD:SW_SPST_B3S-1000" H 4550 6950 50  0001 C CNN
+F 2 "Buttons_Switches_ThroughHole:SW_PUSH_SMALL" H 4550 6950 50  0001 C CNN
 F 3 "" H 4550 6950 50  0000 C CNN
 	1    4550 6750
@@
 F 0 "R4" H 2080 3920 50  0000 L CNN
 F 1 "220R" H 2080 3860 50  0000 L CNN
-F 2 "Resistors_SMD:R_0805" H 2050 3900 50  0001 C CNN
+F 2 "Resistors_ThroughHole:Resistor_Horizontal_RM10mm" H 2050 3900 50  0001 C CNN
 F 3 "" H 2050 3900 50  0000 C CNN
 	1    2050 3900
@@
 Wire Wire Line
 	3100 2650 3100 2450
+$Comp
+L R R10
+U 1 1 5804A9D2
+P 650 3100
+F 0 "R10" V 730 3100 50  0000 C CNN
+F 1 "1M" V 650 3100 50  0000 C CNN
+F 2 "Resistors_ThroughHole:Resistor_Horizontal_RM10mm" V 580 3100 50  0001 C CNN
+F 3 "" H 650 3100 50  0000 C CNN
+	1    650  3100
+	1    0    0    -1
+$EndComp
+$Comp
+L C C3
+U 1 1 5804AA81
+P 1000 3100
+F 0 "C3" H 1025 3200 50  0000 L CNN
+F 1 "4.7nF" H 1025 3000 50  0000 L CNN
+F 2 "Capacitors_ThroughHole:C_Disc_D6_P5" H 1038 2950 50  0001 C CNN
+F 3 "" H 1000 3100 50  0000 C CNN
+	1    1000 3100
+	1    0    0    -1
+$EndComp
+$Comp
+L GND #PWR024
+U 1 1 5804AACA
+P 850 3400
+F 0 "#PWR024" H 850 3150 50  0001 C CNN
+F 1 "GND" H 850 3250 50  0000 C CNN
+F 2 "" H 850 3400 50  0000 C CNN
+F 3 "" H 850 3400 50  0000 C CNN
+	1    850  3400
+	1    0    0    -1
+$EndComp
+Wire Wire Line
+	650  2950 650  2900
+Wire Wire Line
+	650  2900 1000 2900
+Wire Wire Line
+	850  2900 850  2850
+Wire Wire Line
+	1000 2900 1000 2950
+Connection ~ 850  2900
+Wire Wire Line
+	650  3250 650  3300
+Wire Wire Line
+	650  3300 1000 3300
+Wire Wire Line
+	1000 3300 1000 3250
+Wire Wire Line
+	850  3300 850  3400
+Connection ~ 850  3300
 $EndSCHEMATC

Commit message: Added a big decoupling capacitor because of the ESP current glutony
Parts:
- added C4: 150uF, Capacitors_SMD:C_1210_HandSoldering, symbol C_Small
Connections:
- wire segments 85 -> 87
Changed lines of the file:
@@
 LIBS:xilinx
 LIBS:Zilog
-LIBS:esp-01-cache
 EELAYER 25 0
 EELAYER END
@@
 	3700 900  3700 1000
 Wire Wire Line
-	3500 1000 3850 1000
+	3500 1000 4250 1000
 Wire Wire Line
 	3500 1000 3500 1050
@@
 	3500 1250 3500 1350
 Wire Wire Line
-	3500 1350 3850 1350
+	3500 1350 4250 1350
 Wire Wire Line
 	3850 1350 3850 1250
@@
 	850  3300 850  3400
 Connection ~ 850  3300
+$Comp
+L C_Small C4
+U 1 1 580FCE93
+P 4250 1150
+F 0 "C4" H 4260 1220 50  0000 L CNN
+F 1 "150uF" H 4260 1070 50  0000 L CNN
+F 2 "Capacitors_SMD:C_1210_HandSoldering" H 4250 1150 50  0001 C CNN
+F 3 "" H 4250 1150 50  0000 C CNN
+	1    4250 1150
+	1    0    0    -1
+$EndComp
+Wire Wire Line
+	4250 1000 4250 1050
+Connection ~ 3850 1000
+Wire Wire Line
+	4250 1350 4250 1250
+Connection ~ 3850 1350
 $EndSCHEMATC

Commit message: Updated project to follow the kicad official libraries evolutions
Parts:
- SW1, SW2: symbol SW_PUSH_Small_Horizontal -> SW_Push
- U2: symbol LT1761-3.3 -> LT1761-3.3-RESCUE-esp-01
- Y1: symbol CRYSTAL_SMD -> Crystal_GND2
Connections:
- wire segments 87 -> 91
Other:
- moved on the sheet: P1, R9, U1

Commit message: Updated project to follow the kicad official libraries evolutions
Parts:
- C3: footprint Capacitors_ThroughHole:C_Disc_D6_P5 -> Capacitors_THT:C_Disc_D6.0mm_W2.5mm_P5.00mm
- P1: footprint Connect:USB_B -> Connectors:USB_B
- R1, R10, R2, R3, R4, R7, R8: footprint Resistors_ThroughHole:Resistor_Horizontal_RM10mm -> Resistors_THT:R_Axial_DIN0309_L9.0mm_D3.2mm_P12.70mm_Horizontal
- SW1, SW2: footprint Buttons_Switches_ThroughHole:SW_PUSH_SMALL -> Buttons_Switches_THT:SW_PUSH_6mm
Changed lines of the file:
@@
 F 0 "P1" H 1150 2100 50  0000 C CNN
 F 1 "USB_B" H 900 2500 50  0000 C CNN
-F 2 "Connect:USB_B" V 900 2200 50  0001 C CNN
+F 2 "Connectors:USB_B" V 900 2200 50  0001 C CNN
 F 3 "" V 900 2200 50  0000 C CNN
 	1    950  2300
@@
 F 0 "R1" H 2630 2870 50  0000 L CNN
 F 1 "10K" H 2630 2810 50  0000 L CNN
-F 2 "Resistors_ThroughHole:Resistor_Horizontal_RM10mm" H 2600 2850 50  0001 C CNN
+F 2 "Resistors_THT:R_Axial_DIN0309_L9.0mm_D3.2mm_P12.70mm_Horizontal" H 2600 2850 50  0001 C CNN
 F 3 "" H 2600 2850 50  0000 C CNN
 	1    2600 2850
@@
 F 0 "R2" H 1330 3920 50  0000 L CNN
 F 1 "220R" H 1330 3860 50  0000 L CNN
-F 2 "Resistors_ThroughHole:Resistor_Horizontal_RM10mm" H 1300 3900 50  0001 C CNN
+F 2 "Resistors_THT:R_Axial_DIN0309_L9.0mm_D3.2mm_P12.70mm_Horizontal" H 1300 3900 50  0001 C CNN
 F 3 "" H 1300 3900 50  0000 C CNN
 	1    1300 3900
@@
 F 0 "R3" H 1680 3920 50  0000 L CNN
 F 1 "220R" H 1680 3860 50  0000 L CNN
-F 2 "Resistors_ThroughHole:Resistor_Horizontal_RM10mm" H 1650 3900 50  0001 C CNN
+F 2 "Resistors_THT:R_Axial_DIN0309_L9.0mm_D3.2mm_P12.70mm_Horizontal" H 1650 3900 50  0001 C CNN
 F 3 "" H 1650 3900 50  0000 C CNN
 	1    1650 3900
@@
 F 0 "R8" H 8330 4670 50  0000 L CNN
 F 1 "10K" H 8330 4610 50  0000 L CNN
-F 2 "Resistors_ThroughHole:Resistor_Horizontal_RM10mm" H 8300 4650 50  0001 C CNN
+F 2 "Resistors_THT:R_Axial_DIN0309_L9.0mm_D3.2mm_P12.70mm_Horizontal" H 8300 4650 50  0001 C CNN
 F 3 "" H 8300 4650 50  0000 C CNN
 	1    8300 4650
@@
 F 0 "SW2" H 8450 5600 50  0000 C CNN
 F 1 "Bootloader" H 8350 5400 50  0000 L CNN
-F 2 "Buttons_Switches_ThroughHole:SW_PUSH_SMALL" H 8300 5700 50  0001 C CNN
+F 2 "Buttons_Switches_THT:SW_PUSH_6mm" H 8300 5700 50  0001 C CNN
 F 3 "" H 8300 5700 50  0000 C CNN
 	1    8300 5500
@@
 F 0 "R7" H 7830 4670 50  0000 L CNN
 F 1 "10K" H 7830 4610 50  0000 L CNN
-F 2 "Resistors_ThroughHole:Resistor_Horizontal_RM10mm" H 7800 4650 50  0001 C CNN
+F 2 "Resistors_THT:R_Axial_DIN0309_L9.0mm_D3.2mm_P12.70mm_Horizontal" H 7800 4650 50  0001 C CNN
 F 3 "" H 7800 4650 50  0000 C CNN
 	1    7800 4650
@@
 F 0 "SW1" H 4700 6850 50  0000 C CNN
 F 1 "Reset" H 4450 6650 50  0000 L CNN
-F 2 "Buttons_Switches_ThroughHole:SW_PUSH_SMALL" H 4550 6950 50  0001 C CNN
+F 2 "Buttons_Switches_THT:SW_PUSH_6mm" H 4550 6950 50  0001 C CNN
 F 3 "" H 4550 6950 50  0000 C CNN
 	1    4550 6750
@@
 F 0 "R4" H 2080 3920 50  0000 L CNN
 F 1 "220R" H 2080 3860 50  0000 L CNN
-F 2 "Resistors_ThroughHole:Resistor_Horizontal_RM10mm" H 2050 3900 50  0001 C CNN
+F 2 "Resistors_THT:R_Axial_DIN0309_L9.0mm_D3.2mm_P12.70mm_Horizontal" H 2050 3900 50  0001 C CNN
 F 3 "" H 2050 3900 50  0000 C CNN
 	1    2050 3900
@@
 F 0 "R10" V 730 3100 50  0000 C CNN
 F 1 "1M" V 650 3100 50  0000 C CNN
-F 2 "Resistors_ThroughHole:Resistor_Horizontal_RM10mm" V 580 3100 50  0001 C CNN
+F 2 "Resistors_THT:R_Axial_DIN0309_L9.0mm_D3.2mm_P12.70mm_Horizontal" V 580 3100 50  0001 C CNN
 F 3 "" H 650 3100 50  0000 C CNN
 	1    650  3100
@@
 F 0 "C3" H 1025 3200 50  0000 L CNN
 F 1 "4.7nF" H 1025 3000 50  0000 L CNN
-F 2 "Capacitors_ThroughHole:C_Disc_D6_P5" H 1038 2950 50  0001 C CNN
+F 2 "Capacitors_THT:C_Disc_D6.0mm_W2.5mm_P5.00mm" H 1038 2950 50  0001 C CNN
 F 3 "" H 1000 3100 50  0000 C CNN
 	1    1000 3100
